Commit message: cool platform

File: src/dql_multirotor_landing/urdf/moving_platform.urdf (robot description, URDF)
Before this commit: robot moving_platform, 3 links, 2 joints
Links:
- added link moving_platform/wheel_front_left; visual cylinder length=0.1 radius=0.2
- added link moving_platform/wheel_front_right; visual cylinder length=0.1 radius=0.2
- added link moving_platform/wheel_rear_left; visual cylinder length=0.1 radius=0.2
- added link moving_platform/wheel_rear_right; visual cylinder length=0.1 radius=0.2
Joints:
- added joint joint_wheel_front_left: type fixed, parent moving_platform/base_link, child moving_platform/wheel_front_left, origin xyz=0.4 0.55 -0.08 rpy=0 1.57 1.57
- added joint joint_wheel_front_right: type fixed, parent moving_platform/base_link, child moving_platform/wheel_front_right, origin xyz=0.4 -0.55 -0.08 rpy=0 1.57 1.57
- added joint joint_wheel_rear_left: type fixed, parent moving_platform/base_link, child moving_platform/wheel_rear_left, origin xyz=-0.4 0.55 -0.08 rpy=0 1.57 1.57
- added joint joint_wheel_rear_right: type fixed, parent moving_platform/base_link, child moving_platform/wheel_rear_right, origin xyz=-0.4 -0.55 -0.08 rpy=0 1.57 1.57
- joint joint_world_base_link: origin xyz=0 0 0.15 rpy=0 0 0 -> xyz=0 0 0.3 rpy=0 0 0
