Commit message: removed other imu components

File: src/rotors_simulator/rotors_description/urdf/component_snippets.xacro (robot description, xacro)
@@ -233,5 +233,5 @@
   </xacro:macro>
   <!-- Macro to add the controller interface. -->
-  <xacro:macro name="controller_plugin_macro" params="namespace imu_sub_topic">
+  <xacro:macro name="controller_plugin_macro" params="namespace">
     <gazebo>
       <plugin name="controller_interface" filename="librotors_gazebo_controller_interface.so">
@@ -240,5 +240,4 @@
         <commandRateThrustSubTopic>command/rate</commandRateThrustSubTopic>
         <commandMotorSpeedSubTopic>command/motor_speed</commandMotorSpeedSubTopic>
-        <imuSubTopic>${imu_sub_topic}</imuSubTopic>
         <motorSpeedCommandPubTopic>gazebo/command/motor_speed</motorSpeedCommandPubTopic>
       </plugin>
@@ -261,5 +260,5 @@
   <!-- =============================================================== -->
   <xacro:macro name="mavlink_interface_macro"
-    params="namespace mavlink_sub_topic imu_sub_topic mavlink_pub_topic
+    params="namespace mavlink_sub_topic mavlink_pub_topic
       motors_speeds_pub_topic gps_update_freq rotor_count reference_magnetic_field_north
       reference_magnetic_field_east reference_magnetic_field_down reference_latitude
@@ -269,5 +268,4 @@
         <robotNamespace>${namespace}</robotNamespace>
 	<mavlinkControlSubTopic>${mavlink_sub_topic}</mavlinkControlSubTopic>
-        <imuSubTopic>${imu_sub_topic}</imuSubTopic>
         <mavlinkHilSensorPubTopic>${mavlink_pub_topic}</mavlinkHilSensorPubTopic>
 	<motorSpeedsPubTopic>${motors_speeds_pub_topic}</motorSpeedsPubTopic>
@@ -284,45 +282,4 @@
         <referenceLongitude>${reference_longitude}</referenceLongitude> <!-- the initial longitude [degrees [-180, 180]] -->
         <referenceAltitude>${reference_altitude}</referenceAltitude> <!-- the initial altitude [m] -->
-      </plugin>
-    </gazebo>
-  </xacro:macro>
-  <!-- Macro to add an IMU. -->
-  <xacro:macro name="imu_plugin_macro"
-    params="namespace imu_suffix parent_link imu_topic
-      mass_imu_sensor gyroscope_noise_density gyroscope_random_walk
-      gyroscope_bias_correlation_time gyroscope_turn_on_bias_sigma
-      accelerometer_noise_density accelerometer_random_walk
-      accelerometer_bias_correlation_time accelerometer_turn_on_bias_sigma
-      *inertia *origin">
-    <!-- IMU link -->
-    <link name="${namespace}/imu${imu_suffix}_link">
-      <inertial>
-        <xacro:insert_block name="inertia" />
-        <mass value="${mass_imu_sensor}" />  <!-- [kg] -->
-        <origin xyz="0 0 0" rpy="0 0 0" />
-      </inertial>
-    </link>
-    <!-- IMU joint -->
-    <joint name="${namespace}/imu${imu_suffix}_joint" type="revolute">
-      <xacro:insert_block name="origin" />
-      <parent link="${parent_link}" />
-      <child link="${namespace}/imu${imu_suffix}_link" />
-      <limit upper="0" lower="0" effort="0" velocity="0" />
-    </joint>
-    <gazebo>
-      <plugin filename="librotors_gazebo_imu_plugin.so" name="rotors_gazebo_imu${imu_suffix}_plugin">
-      <!-- A good description of the IMU parameters can be found in the kalibr documentation:
-           https://github.com/ethz-asl/kalibr/wiki/IMU-Noise-Model-and-Intrinsics -->
-        <robotNamespace>${namespace}</robotNamespace> <!-- (string, required): ros namespace in which the messages are published -->
-        <linkName>${namespace}/imu${imu_suffix}_link</linkName> <!-- (string, required): name of the body which holds the IMU sensor -->
-        <imuTopic>${imu_topic}</imuTopic> <!-- (string): name of the sensor output topic and prefix of service names (defaults to imu) -->
-        <gyroscopeNoiseDensity>${gyroscope_noise_density}</gyroscopeNoiseDensity> <!-- Gyroscope noise density (two-sided spectrum) [rad/s/sqrt(Hz)] -->
-        <gyroscopeRandomWalk>${gyroscope_random_walk}</gyroscopeRandomWalk> <!-- Gyroscope bias random walk [rad/s/s/sqrt(Hz)] -->
-        <gyroscopeBiasCorrelationTime>${gyroscope_bias_correlation_time}</gyroscopeBiasCorrelationTime> <!-- Gyroscope bias correlation time constant [s] -->
-        <gyroscopeTurnOnBiasSigma>${gyroscope_turn_on_bias_sigma}</gyroscopeTurnOnBiasSigma> <!-- Gyroscope turn on bias standard deviation [rad/s] -->
-        <accelerometerNoiseDensity>${accelerometer_noise_density}</accelerometerNoiseDensity> <!-- Accelerometer noise density (two-sided spectrum) [m/s^2/sqrt(Hz)] -->
-        <accelerometerRandomWalk>${accelerometer_random_walk}</accelerometerRandomWalk> <!-- Accelerometer bias random walk. [m/s^2/s/sqrt(Hz)] -->
-        <accelerometerBiasCorrelationTime>${accelerometer_bias_correlation_time}</accelerometerBiasCorrelationTime> <!-- Accelerometer bias correlation time constant [s] -->
-        <accelerometerTurnOnBiasSigma>${accelerometer_turn_on_bias_sigma}</accelerometerTurnOnBiasSigma> <!-- Accelerometer turn on bias standard deviation [m/s^2] -->
       </plugin>
     </gazebo>
@@ -877,9 +834,8 @@
     </xacro:pressure_sensor_plugin_macro>
   </xacro:macro>
-  <xacro:macro name="default_mavlink_interface" params="namespace imu_sub_topic rotor_count">
+  <xacro:macro name="default_mavlink_interface" params="namespace rotor_count">
     <xacro:mavlink_interface_macro
       namespace="${namespace}"
       mavlink_sub_topic="/mavlink/from"
-      imu_sub_topic="${imu_sub_topic}"
       mavlink_pub_topic="/mavlink/to"
       motors_speeds_pub_topic="gazebo/command/motor_speed"

File: src/rotors_simulator/rotors_description/urdf/hummingbird_base.xacro (robot description, xacro)
@@ -21,14 +21,5 @@
   <xacro:include filename="$(find rotors_description)/urdf/hummingbird.xacro" />
   <!-- Instantiate a controller. -->
-  <xacro:controller_plugin_macro namespace="${namespace}" imu_sub_topic="imu" />
-  <xacro:if value="$(arg enable_mavlink_interface)">
-    <!-- Instantiate mavlink telemetry interface. -->
-    <xacro:default_mavlink_interface namespace="${namespace}" imu_sub_topic="imu" rotor_count="4" />
-  </xacro:if>
-  <!-- Mount an ADIS16448 IMU. -->
-  <!-- <xacro:default_imu namespace="${namespace}" parent_link="${namespace}/base_link" /> -->
-  <!-- <xacro:if value="$(arg enable_ground_truth)">
-    <xacro:ground_truth_imu_and_odometry namespace="${namespace}" parent_link="${namespace}/base_link" />
-  </xacro:if> -->
+  <xacro:controller_plugin_macro namespace="${namespace}" />
   <xacro:if value="$(arg enable_logging)">
     <!-- Instantiate a logger -->
